Commit message: Changed xtion position

File: robots/hera_full.urdf.xacro (robot description, xacro)
@@ -29,4 +29,5 @@
   <xacro:include filename="$(find hera_description)/urdf/simulation/kinect_one.gazebo.xacro" />
   <xacro:include filename="$(find hera_description)/urdf/simulation/manipulator.gazebo.xacro" />
+  <xacro:include filename="$(find hera_description)/urdf/simulation/control.gazebo.xacro" />
 <!-- ####################################################################### -->
 <!-- ######################## robot parts ################################## -->
@@ -59,5 +60,5 @@
     name="xtion"
     parent="torso">
-    <origin xyz="0.1 0 -0.14" rpy="0 0 0" />
+    <origin xyz="0.215 0 -0.17" rpy="0 0 0" />
   </xacro:xtion>
   <!-- torso pointcloud front: kinect_one -->
@@ -80,5 +81,6 @@
   <!-- base -->
   <xacro:gazebo_base
-    reference="base"/>
+    reference="base"
+    update_rate="30"/>
   <!-- hokuyo_utm -->
   <xacro:gazebo_hokuyo_utm
