Commit message: Fixed manipulator limits

File: urdf/actuators/manipulator/manip.urdf.xacro (robot description, xacro)
@@ -56,5 +56,5 @@
       <child link="shoulder_pan_link" />
       <axis xyz="0 0 1" />
-      <limit lower="-3.14" upper="3.14" effort="0" velocity="5" />
+      <limit lower="-1.57" upper="1.57" effort="0" velocity="5" />
     </joint>
   </xacro:macro>
@@ -85,5 +85,5 @@
       <child link="shoulder_lift_link" />
       <axis xyz="0 1 0" />
-      <limit lower="-1.0847" upper="3.14" effort="0" velocity="5" />
+      <limit lower="-0.9" upper="3.55" effort="0" velocity="5" />
     </joint>
   </xacro:macro>
@@ -114,5 +114,5 @@
       <child link="elbow_pan_link" />
       <axis xyz="1 0 0" />
-      <limit lower="-3.14" upper="3.14" effort="0" velocity="5" />
+      <limit lower="-4.71" upper="1.57" effort="0" velocity="5" />
     </joint>
   </xacro:macro>
@@ -143,5 +143,5 @@
       <child link="elbow_lift_link" />
       <axis xyz="0 -1 0" />
-      <limit lower="-3.14" upper="1.0078" effort="0" velocity="5" />
+      <limit lower="-4" upper="1.0078" effort="0" velocity="5" />
     </joint>
   </xacro:macro>
@@ -201,5 +201,5 @@
       <child link="wrist_lift_link" />
       <axis xyz="0 -1 0" />
-      <limit lower="-2.6232" upper="1.8262" effort="0" velocity="5" />
+      <limit lower="-0.64" upper="4" effort="0" velocity="5" />
     </joint>
   </xacro:macro>

File: urdf/actuators/torso.urdf.xacro (robot description, xacro)
@@ -105,5 +105,5 @@
       <parent link="${name}"/>
       <child link="${name}_sensor_plat"/>
-      <axis xyz="0 1 0"/>
+      <axis xyz="0 -1 0"/>
       <limit effort="${torso_sensor_plat_effort}" velocity="${torso_sensor_plat_velocity}"
         lower="0.0" upper="${M_PI/2}"/>
