Commit message: ros2

File: urdf/actuators/base.urdf.xacro (robot description, xacro)
@@ -52,5 +52,5 @@
         <material name="black"/>
         <geometry>
-          <mesh filename="package://hera_description/meshes/base.stl"/>
+          <mesh filename="file://$(find hera_description)/meshes/base.stl"/>
         </geometry>
       </visual>
@@ -65,5 +65,5 @@
         <material name="white"/>
         <geometry>
-          <mesh filename="package://hera_description/meshes/wheelF.stl"/>
+          <mesh filename="file://$(find hera_description)/meshes/wheelF.stl"/>
         </geometry>
       </visual>
@@ -78,5 +78,5 @@
         <material name="white"/>
         <geometry>
-          <mesh filename="package://hera_description/meshes/wheelF.stl"/>
+          <mesh filename="file://$(find hera_description)/meshes/wheelF.stl"/>
         </geometry>
       </visual>
@@ -91,5 +91,5 @@
         <material name="white"/>
         <geometry>
-          <mesh filename="package://hera_description/meshes/wheelB.stl"/>
+          <mesh filename="file://$(find hera_description)/meshes/wheelB.stl"/>
         </geometry>
       </visual>
@@ -104,5 +104,5 @@
         <material name="white"/>
         <geometry>
-          <mesh filename="package://hera_description/meshes/wheelB.stl"/>
+          <mesh filename="file://$(find hera_description)/meshes/wheelB.stl"/>
         </geometry>
       </visual>

File: urdf/actuators/head.urdf.xacro (robot description, xacro)
@@ -49,5 +49,5 @@
         <material name="grey"/>
         <geometry>
-          <mesh filename="package://hera_description/meshes/head.stl"/>
+          <mesh filename="file://$(find hera_description)/meshes/head.stl"/>
         </geometry>
       </visual>

File: urdf/actuators/manipulator/manip.urdf.xacro (robot description, xacro)
@@ -8,13 +8,13 @@
         <origin xyz="0 0 0" rpy="0 0 0" />
         <geometry>
-          <mesh filename="package://hera_description/meshes/manip_meshes/manip_base.STL"/>
-        </geometry>
-        <material name="dark_grey">
-        </material>
-      </visual>
-      <collision>
-        <origin xyz="0 0 0" rpy="0 0 0" />
-        <geometry>
-          <mesh filename="package://hera_description/meshes/manip_meshes/manip_base_col.STL"/>
+          <mesh filename="file://$(find hera_description)/meshes/manip_meshes/manip_base.STL"/>
+        </geometry>
+        <material name="dark_grey">
+        </material>
+      </visual>
+      <collision>
+        <origin xyz="0 0 0" rpy="0 0 0" />
+        <geometry>
+          <mesh filename="file://$(find hera_description)/meshes/manip_meshes/manip_base_col.STL"/>
         </geometry>
       </collision>
@@ -36,5 +36,5 @@
         <origin xyz="0 0 0" rpy="0 0 0" />
         <geometry>
-          <mesh filename="package://hera_description/meshes/manip_meshes/shoulder_pan.STL"/>
+          <mesh filename="file://$(find hera_description)/meshes/manip_meshes/shoulder_pan.STL"/>
         </geometry>
         <material name="dark_grey">
@@ -45,5 +45,5 @@
         <origin xyz="0 0 0" rpy="0 0 0" />
         <geometry>
-          <mesh filename="package://hera_description/meshes/manip_meshes/shoulder_pan_col.STL"/>
+          <mesh filename="file://$(find hera_description)/meshes/manip_meshes/shoulder_pan_col.STL"/>
         </geometry>
       </collision>
@@ -65,14 +65,14 @@
         <origin xyz="0 0 0" rpy="0 0 0" />
         <geometry>
-          <mesh filename="package://hera_description/meshes/manip_meshes/shoulder_lift.STL"/>
-        </geometry>
-        <material name="dark_grey">
-          <color rgba="0.898039215686275 0.917647058823529 0.929411764705882 1" />
-        </material>
-      </visual>
-      <collision>
-        <origin xyz="0 0 0" rpy="0 0 0" />
-        <geometry>
-          <mesh filename="package://hera_description/meshes/manip_meshes/shoulder_lift_col.STL"/>
+          <mesh filename="file://$(find hera_description)/meshes/manip_meshes/shoulder_lift.STL"/>
+        </geometry>
+        <material name="dark_grey">
+          <color rgba="0.898039215686275 0.917647058823529 0.929411764705882 1" />
+        </material>
+      </visual>
+      <collision>
+        <origin xyz="0 0 0" rpy="0 0 0" />
+        <geometry>
+          <mesh filename="file://$(find hera_description)/meshes/manip_meshes/shoulder_lift_col.STL"/>
         </geometry>
       </collision>
@@ -94,5 +94,5 @@
         <origin xyz="0 0 0" rpy="0 0 0" />
         <geometry>
-          <mesh filename="package://hera_description/meshes/manip_meshes/elbow_pan.STL"/>
+          <mesh filename="file://$(find hera_description)/meshes/manip_meshes/elbow_pan.STL"/>
         </geometry>
         <material name="dark_grey">
@@ -103,5 +103,5 @@
         <origin xyz="0 0 0" rpy="0 0 0" />
         <geometry>
-          <mesh filename="package://hera_description/meshes/manip_meshes/elbow_pan_col.STL"/>
+          <mesh filename="file://$(find hera_description)/meshes/manip_meshes/elbow_pan_col.STL"/>
         </geometry>
       </collision>
@@ -123,14 +123,14 @@
         <origin xyz="0 0 0" rpy="0 0 0" />
         <geometry>
-          <mesh filename="package://hera_description/meshes/manip_meshes/elbow_lift.STL"/>
-        </geometry>
-        <material name="dark_grey">
-          <color rgba="0.898039215686275 0.917647058823529 0.929411764705882 1" />
-        </material>
-      </visual>
-      <collision>
-        <origin xyz="0 0 0" rpy="0 0 0" />
-        <geometry>
-          <mesh filename="package://hera_description/meshes/manip_meshes/elbow_lift_col.STL"/>
+          <mesh filename="file://$(find hera_description)/meshes/manip_meshes/elbow_lift.STL"/>
+        </geometry>
+        <material name="dark_grey">
+          <color rgba="0.898039215686275 0.917647058823529 0.929411764705882 1" />
+        </material>
+      </visual>
+      <collision>
+        <origin xyz="0 0 0" rpy="0 0 0" />
+        <geometry>
+          <mesh filename="file://$(find hera_description)/meshes/manip_meshes/elbow_lift_col.STL"/>
         </geometry>
       </collision>
@@ -152,5 +152,5 @@
         <origin xyz="0 0 0" rpy="0 0 0"/>
         <geometry>
-          <mesh  filename="package://hera_description/meshes/manip_meshes/wrist_pan.STL" />
+          <mesh  filename="file://$(find hera_description)/meshes/manip_meshes/wrist_pan.STL" />
         </geometry>
         <material name="dark_grey">
@@ -161,5 +161,5 @@
         <origin xyz="0 0 0" rpy="0 0 0"/>
         <geometry>
-          <mesh filename="package://hera_description/meshes/manip_meshes/wrist_pan_col.STL" />
+          <mesh filename="file://$(find hera_description)/meshes/manip_meshes/wrist_pan_col.STL" />
         </geometry>
       </collision>
@@ -181,5 +181,5 @@
         <origin xyz="0 0 0" rpy="0 0 0"/>
         <geometry>
-          <mesh  filename="package://hera_description/meshes/manip_meshes/wrist_lift.STL" />
+          <mesh  filename="file://$(find hera_description)/meshes/manip_meshes/wrist_lift.STL" />
         </geometry>
         <material name="dark_grey">
@@ -190,5 +190,5 @@
         <origin xyz="0 0 0" rpy="0 0 0"/>
         <geometry>
-          <mesh filename="package://hera_description/meshes/manip_meshes/wrist_lift_col.STL" />
+          <mesh filename="file://$(find hera_description)/meshes/manip_meshes/wrist_lift_col.STL" />
         </geometry>
         </collision>
@@ -210,14 +210,14 @@
         <origin xyz="0 0 0" rpy="0 0 0" />
         <geometry>
-          <mesh filename="package://hera_description/meshes/manip_meshes/gripper_meshes/gripper_right.STL"/>
-        </geometry>
-        <material name="dark_grey">
-          <color rgba="0.898039215686275 0.917647058823529 0.929411764705882 1" />
-        </material>
-      </visual>
-      <collision>
-        <origin xyz="0 0 0" rpy="0 0 0" />
-        <geometry>
-          <mesh filename="package://hera_description/meshes/manip_meshes/gripper_meshes/gripper_right_col.STL"/>
+          <mesh filename="file://$(find hera_description)/meshes/manip_meshes/gripper_meshes/gripper_right.STL"/>
+        </geometry>
+        <material name="dark_grey">
+          <color rgba="0.898039215686275 0.917647058823529 0.929411764705882 1" />
+        </material>
+      </visual>
+      <collision>
+        <origin xyz="0 0 0" rpy="0 0 0" />
+        <geometry>
+          <mesh filename="file://$(find hera_description)/meshes/manip_meshes/gripper_meshes/gripper_right_col.STL"/>
         </geometry>
       </collision>
@@ -239,5 +239,5 @@
         <origin xyz="0 0 0" rpy="0 0 0" />
         <geometry>
-          <mesh filename="package://hera_description/meshes/manip_meshes/gripper_meshes/gripper_right_end.STL"/>
+          <mesh filename="file://$(find hera_description)/meshes/manip_meshes/gripper_meshes/gripper_right_end.STL"/>
         </geometry>
         <material name="white">
@@ -248,5 +248,5 @@
         <origin xyz="0 0 0" rpy="0 0 0" />
         <geometry>
-          <mesh filename="package://hera_description/meshes/manip_meshes/gripper_meshes/gripper_right_end.STL"/>
+          <mesh filename="file://$(find hera_description)/meshes/manip_meshes/gripper_meshes/gripper_right_end.STL"/>
         </geometry>
       </collision>
@@ -267,14 +267,14 @@
         <origin xyz="0 0 0" rpy="0 0 0" />
         <geometry>
-          <mesh filename="package://hera_description/meshes/manip_meshes/gripper_meshes/gripper_left.STL" />
-        </geometry>
-        <material name="dark_grey">
-          <color rgba="0.898039215686275 0.917647058823529 0.929411764705882 1" />
-        </material>
-      </visual>
-      <collision>
-        <origin xyz="0 0 0" rpy="0 0 0" />
-        <geometry>
-          <mesh filename="package://hera_description/meshes/manip_meshes/gripper_meshes/gripper_left.STL" />
+          <mesh filename="file://$(find hera_description)/meshes/manip_meshes/gripper_meshes/gripper_left.STL" />
+        </geometry>
+        <material name="dark_grey">
+          <color rgba="0.898039215686275 0.917647058823529 0.929411764705882 1" />
+        </material>
+      </visual>
+      <collision>
+        <origin xyz="0 0 0" rpy="0 0 0" />
+        <geometry>
+          <mesh filename="file://$(find hera_description)/meshes/manip_meshes/gripper_meshes/gripper_left.STL" />
         </geometry>
       </collision>
@@ -296,5 +296,5 @@
         <origin xyz="0 0 0" rpy="0 0 0" />
         <geometry>
-          <mesh filename="package://hera_description/meshes/manip_meshes/gripper_meshes/gripper_left_end.STL" />
+          <mesh filename="file://$(find hera_description)/meshes/manip_meshes/gripper_meshes/gripper_left_end.STL" />
         </geometry>
         <material name="white">
@@ -305,5 +305,5 @@
         <origin xyz="0 0 0" rpy="0 0 0" />
         <geometry>
-          <mesh filename="package://hera_description/meshes/manip_meshes/gripper_meshes/gripper_left_end.STL" />
+          <mesh filename="file://$(find hera_description)/meshes/manip_meshes/gripper_meshes/gripper_left_end.STL" />
         </geometry>
       </collision>

File: urdf/actuators/torso.urdf.xacro (robot description, xacro)
@@ -68,5 +68,5 @@
         <material name="dark_grey"/>
         <geometry>
-          <mesh filename="package://hera_description/meshes/torso.stl"/>
+          <mesh filename="file://$(find hera_description)/meshes/torso.stl"/>
         </geometry>
       </visual>
@@ -75,5 +75,5 @@
         <material name="dark_grey"/>
         <geometry>
-          <mesh filename="package://hera_description/meshes/torso.stl"/>
+          <mesh filename="file://$(find hera_description)/meshes/torso.stl"/>
         </geometry>
       </collision>
@@ -92,5 +92,5 @@
         <material name="dark_grey"/>
         <geometry>
-          <mesh filename="package://hera_description/meshes/torso_sensor_plat.stl"/>
+          <mesh filename="file://$(find hera_description)/meshes/torso_sensor_plat.stl"/>
         </geometry>
       </visual>
@@ -126,5 +126,5 @@
         <origin xyz="0 0 0" rpy="0 0 0" />
         <geometry>
-          <mesh filename="package://hera_description/meshes/manip_meshes/manip_support.STL"/>
+          <mesh filename="file://$(find hera_description)/meshes/manip_meshes/manip_support.STL"/>
         </geometry>
         <material name="grey">
@@ -135,5 +135,5 @@
         <origin xyz="0 0 0" rpy="0 0 0" />
         <geometry>
-          <mesh filename="package://hera_description/meshes/manip_meshes/manip_support.STL"/>
+          <mesh filename="file://$(find hera_description)/meshes/manip_meshes/manip_support.STL"/>
         </geometry>
       </collision>
@@ -155,5 +155,5 @@
         <origin xyz="0 0 0" rpy="0 0 0" />
         <geometry>
-          <mesh filename="package://hera_description/meshes/manip_meshes/backrest.STL"/>
+          <mesh filename="file://$(find hera_description)/meshes/manip_meshes/backrest.STL"/>
         </geometry>
         <material name="grey">
@@ -164,5 +164,5 @@
         <origin xyz="0 0 0" rpy="0 0 0" />
         <geometry>
-          <mesh filename="package://hera_description/meshes/manip_meshes/backrest.STL"/>
+          <mesh filename="file://$(find hera_description)/meshes/manip_meshes/backrest.STL"/>
         </geometry>
       </collision>

File: urdf/sensors/asus_xtion.urdf.xacro (robot description, xacro)
@@ -18,5 +18,5 @@
         <origin xyz="0.02 0.025 0" rpy="${M_PI/2} 0.0 ${M_PI/2}" />
         <geometry>
-          <mesh filename="package://hera_description/meshes/asus_xtion.stl"/>
+          <mesh filename="file://$(find hera_description)/meshes/asus_xtion.stl"/>
         </geometry>
       </visual>

File: urdf/sensors/hokuyo_urg.urdf.xacro (robot description, xacro)
@@ -17,5 +17,5 @@
         <origin xyz="0 0 0" rpy="0 0 0" />
         <geometry>
-          <mesh filename="package://hera_description/meshes/hokuyo_urg.dae" />
+          <mesh filename="file://$(find hera_description)/meshes/hokuyo_urg.dae" />
         </geometry>
       </visual>

File: urdf/sensors/hokuyo_utm.urdf.xacro (robot description, xacro)
@@ -17,5 +17,5 @@
         <origin xyz="0 0 0" rpy="${M_PI/2} 0 0" />
         <geometry>
-          <mesh filename="package://hera_description/meshes/hokuyo_utm.stl"/>
+          <mesh filename="file://$(find hera_description)/meshes/hokuyo_utm.stl"/>
         </geometry>
       </visual>

File: urdf/sensors/kinect_one.urdf.xacro (robot description, xacro)
@@ -18,5 +18,5 @@
         <origin xyz="0 -0.01 0" rpy="0.0 0.0 0.0" />
         <geometry>
-          <mesh filename="package://hera_description/meshes/kinect_one.stl"/>
+          <mesh filename="file://$(find hera_description)/meshes/kinect_one.stl"/>
         </geometry>
       </visual>
